Commit message: visual servoing simulationr results

File: franka_panda/franka_ros/franka_description/robots/panda_arm_camera.urdf.xacro (robot description, xacro)
@@ -5,5 +5,8 @@
   <xacro:include filename="$(find franka_description)/robots/panda_arm_hand.effort.urdf.xacro"/>
   <xacro:include filename="$(find franka_description)/robots/depth.xacro" />
-  <xacro:camera_gazebo_sensor xyz="0.06 -0.00 0" rpy="-1.57 -1.57 0.0"
+  <!-- <xacro:camera_gazebo_sensor xyz="0.06 -0.00 0.0" rpy="-1.57 -1.57 -0.77"
+			      parent="panda_link8"
+			      sensor_name="panda_camera" /> -->
+  <xacro:camera_gazebo_sensor xyz="0.06 -0.00 0.0" rpy="-1.57 -1.57 0.0"
 			      parent="panda_link8"
 			      sensor_name="panda_camera" />

File: toy_problem/urdf/vbmbot.xacro (robot description, xacro)
@@ -114,5 +114,5 @@
   <joint name="camera_joint" type="fixed">
     <!--<axis xyz="0 0 0" /> -->
-    <origin xyz="${camera_link} 0 ${height3 - axel_offset}" rpy="0 0 0 "/>
+    <origin xyz="0 0 ${height3 - axel_offset}" rpy="0 0 0 "/>
     <parent link="link3"/>
     <child link="camera_link"/>
